Commit message: Workingish hardware path

File: lk_description/urdf/rover.urdf (robot description, URDF)
Before this commit: robot sirdigsalot, 7 links, 6 joints
Joints:
- removed joint base_to_left_back_wheel
- removed joint base_to_left_front_wheel
- removed joint base_to_right_back_wheel
- removed joint base_to_right_front_wheel
- added joint bl_wheel_joint: type continuous, parent base_link, child left_back_wheel, origin xyz=-.2667 -.365125 0, axis 1 0 0
- added joint br_wheel_joint: type continuous, parent base_link, child right_back_wheel, origin xyz=.2667 -.365125 0, axis 1 0 0
- added joint lf_wheel_joint: type continuous, parent base_link, child left_front_wheel, origin xyz=-.2667 .365125 0, axis 1 0 0
- added joint rf_wheel_joint: type continuous, parent base_link, child right_front_wheel, origin xyz=.2667 .365125 0, axis 1 0 0

Commit message: Working URDF file

File: lk_description/urdf/rover.urdf (robot description, URDF)
Before this commit: robot sirdigsalot, 7 links, 6 joints
Joints:
- removed joint bl_wheel_joint
- removed joint br_wheel_joint
- added joint lb_wheel_joint: type continuous, parent base_link, child left_back_wheel, origin xyz=-.2667 -.365125 0, axis 1 0 0
- added joint rb_wheel_joint: type continuous, parent base_link, child right_back_wheel, origin xyz=.2667 -.365125 0, axis 1 0 0
