Commit message: Update Code to work with Simulator & Diff drive

File: lk_description/urdf/model.xacro (robot description, xacro)
@@ -1,4 +1,9 @@
 <robot
   name="sirdigsalot">
+  <!-- <link name="world"/> -->
+  <!-- <joint name="fixed" type="fixed">
+    <parent link="world"/>
+    <child link="base_link"/>
+  </joint> -->
   <link
     name="base_link">
@@ -62,20 +67,22 @@
         rpy="0 0 0" />
       <geometry>
-        <mesh
-          filename="package://lk_description/meshes/frontLeftWheel.STL" />
-      </geometry>
-      <material
-        name="">
-        <color
-          rgba="0.79216 0.81961 0.93333 1" />
-      </material>
-    </visual>
-    <collision>
-      <origin
-        xyz="0 0 0"
-        rpy="0 0 0" />
-      <geometry>
-        <mesh
-          filename="package://lk_description/meshes/frontLeftWheel.STL" />
+          <cylinder length=".1016" radius=".1524"/>
+        <!-- <mesh
+          filename="package://lk_description/meshes/frontLeftWheel.STL" /> -->
+      </geometry>
+      <material
+        name="">
+        <color
+          rgba="0.79216 0.81961 0.93333 1" />
+      </material>
+    </visual>
+    <collision>
+      <origin
+        xyz="0 0 0"
+        rpy="0 0 0" />
+      <geometry>
+        <!-- <mesh
+          filename="package://lk_description/meshes/frontLeftWheel.STL" /> -->
+        <cylinder length=".1016" radius=".1524"/>
       </geometry>
     </collision>
@@ -115,20 +122,22 @@
         rpy="0 0 0" />
       <geometry>
-        <mesh
-          filename="package://lk_description/meshes/backLeftWheel.STL" />
-      </geometry>
-      <material
-        name="">
-        <color
-          rgba="0.79216 0.81961 0.93333 1" />
-      </material>
-    </visual>
-    <collision>
-      <origin
-        xyz="0 0 0"
-        rpy="0 0 0" />
-      <geometry>
-        <mesh
-          filename="package://lk_description/meshes/backLeftWheel.STL" />
+        <!-- <mesh
+          filename="package://lk_description/meshes/backLeftWheel.STL" /> -->
+                  <cylinder length=".1016" radius=".1524"/>
+      </geometry>
+      <material
+        name="">
+        <color
+          rgba="0.79216 0.81961 0.93333 1" />
+      </material>
+    </visual>
+    <collision>
+      <origin
+        xyz="0 0 0"
+        rpy="0 0 0" />
+      <geometry>
+        <!-- <mesh
+          filename="package://lk_description/meshes/backLeftWheel.STL" /> -->
+                  <cylinder length=".1016" radius=".1524"/>
       </geometry>
     </collision>
@@ -168,20 +177,22 @@
         rpy="0 0 0" />
       <geometry>
-        <mesh
-          filename="package://lk_description/meshes/frontRightWheel.STL" />
-      </geometry>
-      <material
-        name="">
-        <color
-          rgba="0.79216 0.81961 0.93333 1" />
-      </material>
-    </visual>
-    <collision>
-      <origin
-        xyz="0 0 0"
-        rpy="0 0 0" />
-      <geometry>
-        <mesh
-          filename="package://lk_description/meshes/frontRightWheel.STL" />
+        <!-- <mesh
+          filename="package://lk_description/meshes/frontRightWheel.STL" /> -->
+                  <cylinder length=".1016" radius=".1524"/>
+      </geometry>
+      <material
+        name="">
+        <color
+          rgba="0.79216 0.81961 0.93333 1" />
+      </material>
+    </visual>
+    <collision>
+      <origin
+        xyz="0 0 0"
+        rpy="0 0 0" />
+      <geometry>
+        <!-- <mesh
+          filename="package://lk_description/meshes/frontRightWheel.STL" /> -->
+                  <cylinder length=".1016" radius=".1524"/>
       </geometry>
     </collision>
@@ -221,6 +232,7 @@
         rpy="0 0 0" />
       <geometry>
-        <mesh
-          filename="package://lk_description/meshes/backRightWheel.STL" />
+        <!-- <mesh
+          filename="package://lk_description/meshes/backRightWheel.STL" /> -->
+                  <cylinder length=".1016" radius=".1524"/>
       </geometry>
       <material
@@ -235,6 +247,7 @@
         rpy="0 0 0" />
       <geometry>
-        <mesh
-          filename="package://lk_description/meshes/backRightWheel.STL" />
+        <!-- <mesh
+          filename="package://lk_description/meshes/backRightWheel.STL" /> -->
+                  <cylinder length=".1016" radius=".1524"/>
       </geometry>
     </collision>
@@ -253,5 +266,5 @@
       xyz="0 0 1" />
   </joint>
-  <link
+  <!-- <link
     name="depRightActuator">
     <inertial>
@@ -292,6 +305,6 @@
       </geometry>
     </collision>
-  </link>
-  <joint
+  </link> -->
+  <!-- <joint
     name="depRightExtend"
     type="prismatic">
@@ -531,4 +544,50 @@
       effort="0"
       velocity="0" />
-  </joint>
-</robot>
+  </joint> -->
+    <gazebo>
+    <plugin name="gazebo_ros_control" filename="libgazebo_ros_control.so">
+      <robotNamespace>/sirdigsalot</robotNamespace>
+      <!-- <robotParam>/robot_description</robotParam> -->
+      <robotSimType>gazebo_ros_control/DefaultRobotHWSim</robotSimType>
+    </plugin>
+  </gazebo>
+		<transmission name="backLeftWheelTrans" type="SimpleTransmission">
+			<type>transmission_interface/SimpleTransmission</type>
+			<actuator name="backLeftWheelMotor">
+				<mechanicalReduction>1</mechanicalReduction>
+        <hardwareInterface>VelocityJointInterface</hardwareInterface>
+			</actuator>
+			<joint name="backLeftWheelRotate">
+				<hardwareInterface>hardware_interface/VelocityJointInterface</hardwareInterface>
+			</joint>
+		</transmission>
+		<transmission name="frontLeftWheelTrans" type="SimpleTransmission">
+			<type>transmission_interface/SimpleTransmission</type>
+			<actuator name="frontLeftWheelMotor">
+				<mechanicalReduction>1</mechanicalReduction>
+        <hardwareInterface>VelocityJointInterface</hardwareInterface>
+			</actuator>
+			<joint name="frontLeftWheelRotate">
+				<hardwareInterface>hardware_interface/VelocityJointInterface</hardwareInterface>
+			</joint>
+		</transmission>
+		<transmission name="backRightWheelTrans" type="SimpleTransmission">
+			<type>transmission_interface/SimpleTransmission</type>
+			<actuator name="backRightWheelMotor">
+				<mechanicalReduction>1</mechanicalReduction>
+        <hardwareInterface>VelocityJointInterface</hardwareInterface>
+			</actuator>
+			<joint name="backRightWheelRotate">
+				<hardwareInterface>hardware_interface/VelocityJointInterface</hardwareInterface>
+			</joint>
+		</transmission>
+		<transmission name="frontRightWheelTrans" type="SimpleTransmission">
+			<type>transmission_interface/SimpleTransmission</type>
+			<actuator name="frontRightWheelMotor">
+				<mechanicalReduction>1</mechanicalReduction>
+        <hardwareInterface>VelocityJointInterface</hardwareInterface>
+			</actuator>
+			<joint name="frontRightWheelRotate">
+				<hardwareInterface>hardware_interface/VelocityJointInterface</hardwareInterface>
+			</joint>
+		</transmission>
